Commit message: fix:fix the readme

File: car_total/urdf/car_total.urdf (robot description, URDF)
Before this commit: robot car_total, 17 links, 16 joints
Joints:
- joint left_ahead_arm_joint: limit lower=-2.356 upper=2.356 effort=50 velocity=1.57 -> lower=-0.523 upper=3.926 effort=50 velocity=1.57
- joint left_back_arm_joint: limit lower=-2.356 upper=2.356 effort=50 velocity=1.57 -> lower=-3.926 upper=0.523 effort=50 velocity=1.57
- joint right_ahead_arm_joint: limit lower=-2.356 upper=2.356 effort=50 velocity=1.57 -> lower=-0.523 upper=3.926 effort=50 velocity=1.57
- joint right_back_arm_joint: limit lower=-2.356 upper=2.356 effort=50 velocity=1.57 -> lower=-3.926 upper=0.523 effort=50 velocity=1.57
