Commit message: fix: use ascii car_urdf identifiers

File: car_urdf/urdf/car24.urdf (robot description, URDF)
Before this commit: robot 四摆臂六履带, 18 links, 17 joints
Links:
- link base_link: geometry collision mesh filename=package://car_urdf/meshes/base_link.STL; visual mesh filename=package://car_urdf/meshes/base_link.STL
- link camera_link: geometry collision mesh filename=package://car_urdf/meshes/camera_link.STL; visual mesh filename=package://car_urdf/meshes/camera_link.STL
- link catch_camera: geometry collision mesh filename=package://car_urdf/meshes/catch_camera.STL; visual mesh filename=package://car_urdf/meshes/catch_camera.STL
- link end_effector_link: geometry collision mesh filename=package://car_urdf/meshes/end_effector_link.STL; visual mesh filename=package://car_urdf/meshes/end_effector_link.STL
- link forearm_link: geometry collision mesh filename=package://car_urdf/meshes/forearm_link.STL; visual mesh filename=package://car_urdf/meshes/forearm_link.STL
- link front_left_flipper_link: geometry collision mesh filename=package://car_urdf/meshes/front_left_flipper_link.STL; visual mesh filename=package://car_urdf/meshes/front_left_flipper_link.STL
- link front_left_track_driver_link: geometry collision mesh filename=package://car_urdf/meshes/front_left_track_driver_link.STL; visual mesh filename=package://car_urdf/meshes/front_left_track_driver_link.STL
- link front_right_flipper_link: geometry collision mesh filename=package://car_urdf/meshes/front_right_flipper_link.STL; visual mesh filename=package://car_urdf/meshes/front_right_flipper_link.STL
- link front_right_track_driver_link: geometry collision mesh filename=package://car_urdf/meshes/front_right_track_driver_link.STL; visual mesh filename=package://car_urdf/meshes/front_right_track_driver_link.STL
- link lidar_link: geometry collision mesh filename=package://car_urdf/meshes/lidar_link.STL; visual mesh filename=package://car_urdf/meshes/lidar_link.STL
- link rear_left_flipper_link: geometry collision mesh filename=package://car_urdf/meshes/rear_left_flipper_link.STL; visual mesh filename=package://car_urdf/meshes/rear_left_flipper_link.STL
- link rear_left_track_driver_link: geometry collision mesh filename=package://car_urdf/meshes/rear_left_track_driver_link.STL; visual mesh filename=package://car_urdf/meshes/rear_left_track_driver_link.STL
- link rear_right_flipper_link: geometry collision mesh filename=package://car_urdf/meshes/rear_right_flipper_link.STL; visual mesh filename=package://car_urdf/meshes/rear_right_flipper_link.STL
- link rear_right_track_driver_link: geometry collision mesh filename=package://car_urdf/meshes/rear_right_track_driver_link.STL; visual mesh filename=package://car_urdf/meshes/rear_right_track_driver_link.STL
- link turret_link: geometry collision mesh filename=package://car_urdf/meshes/turret_link.STL; visual mesh filename=package://car_urdf/meshes/turret_link.STL
- link upper_arm_link: geometry collision mesh filename=package://car_urdf/meshes/upper_arm_link.STL; visual mesh filename=package://car_urdf/meshes/upper_arm_link.STL
- link wrist_pitch_link: geometry collision mesh filename=package://car_urdf/meshes/wrist_pitch_link.STL; visual mesh filename=package://car_urdf/meshes/wrist_pitch_link.STL
- link wrist_roll_link: geometry collision mesh filename=package://car_urdf/meshes/wrist_roll_link.STL; visual mesh filename=package://car_urdf/meshes/wrist_roll_link.STL
