Commit message: car_urdf: normalize joints, sync limits, and fix root link warning

File: car_urdf/urdf/car_urdf.urdf (robot description, URDF)
Before this commit: robot car_urdf, 18 links, 17 joints
Links:
- added link base_link_root
- added link zhua1, mass 0.0276512162867833; collision box size=0.001 0.0005 0.0025; visual mesh filename=package://car_urdf/meshes/zhua1.STL
- added link zhua2, mass 0.0276512162867832; collision box size=0.001 0.0005 0.0025; visual mesh filename=package://car_urdf/meshes/zhua2.STL
- link camera: mass 0.0491654266514404 -> 0.0491654266514403
- link catch_camera: mass 1.07678794206715 -> 0.05; geometry visual mesh filename=package://car_urdf/meshes/catch_camera.STL
- link handshands_course_part: mass 0.229769688817791 -> 0.174467256244225; geometry collision cylinder length=0.08 radius=0.02; visual mesh filename=package://car_urdf/meshes/handshands_course_part.STL
- link small_pitch_part: mass 1.16129891011757 -> 1.16129891011756
Joints:
- removed joint big_course_joint
- removed joint big_pitch_joint
- removed joint catch_camera
- removed joint hands_course_joint
- removed joint hands_pitch_joint
- removed joint hands_roll_joint
- removed joint left_ahead_arm_joint
- removed joint left_ahead_wheel_joint
- removed joint left_back_arm_joint
- removed joint left_back_wheel_joint
- removed joint right_ahead_arm_joint
- removed joint right_ahead_wheel_joint
- removed joint right_back_arm_joint
- removed joint right_back_wheel_joint
- removed joint small_pitch_joint
- added joint base_link_root_joint: type fixed, parent base_link_root, child base_link, origin xyz=0 0 0 rpy=0 0 0
- added joint elbow_pitch_joint: type revolute, parent big_pitch_part, child small_pitch_part, origin xyz=0 -0.00980000000004102 0.515300000000048 rpy=0 0 0, axis 0 -1 0, limit lower=-1.0 upper=2.793 effort=18 velocity=1.57
- added joint gripper_camera_mount_joint: type fixed, parent handshands_course_part, child catch_camera, origin xyz=-0.0462233943895681 0.00134448857148927 0.0777106538096684 rpy=0 0 0
- added joint left_front_arm_joint: type revolute, parent base_link, child left_ahead_arm, origin xyz=-0.277600000000002 -0.241000195879134 0.0551000000000096 rpy=0 0 0, axis 0 -1 0, limit lower=-3.665 upper=0.524 effort=50 velocity=1.57
- added joint left_front_wheel_joint: type continuous, parent base_link, child left_ahead_wheel, origin xyz=-0.155999999999997 -0.219000195879134 0 rpy=0 0 0, axis 0 1 0
- added joint left_gripper_finger_joint: type prismatic, parent handshands_course_part, child zhua1, origin xyz=0 0.021924 0.0985 rpy=0 0 0, axis 0 1 0, limit lower=-0.022 upper=0.03 effort=1 velocity=3
- added joint left_rear_arm_joint: type revolute, parent base_link, child left_back_arm, origin xyz=0.277599999999999 -0.241000195879128 0.0551000000000025 rpy=0 0 0, axis 0 -1 0, limit lower=-0.524 upper=3.665 effort=50 velocity=1.57
- added joint left_rear_wheel_joint: type continuous, parent base_link, child left_back_wheel, origin xyz=0.156000000000004 -0.219000195879131 0 rpy=0 0 0, axis 0 1 0
- added joint right_front_arm_joint: type revolute, parent base_link, child right_ahead_arm, origin xyz=-0.277600000000005 0.24100019587914 0.0551000000000029 rpy=0 0 0, axis 0 1 0, limit lower=-3.665 upper=0.524 effort=50 velocity=1.57
- added joint right_front_wheel_joint: type continuous, parent base_link, child right_ahead_wheel, origin xyz=-0.155999999999997 0.219000195879134 0 rpy=0 0 0, axis 0 1 0
- added joint right_gripper_finger_joint: type prismatic, parent handshands_course_part, child zhua2, origin xyz=-0.0038322 -0.021924 0.0985 rpy=0 0 0, axis 0 -1 0, limit lower=-0.022 upper=0.03 effort=1 velocity=3, mimic joint=left_gripper_finger_joint multiplier=1 offset=0
- added joint right_rear_arm_joint: type revolute, parent base_link, child right_back_arm, origin xyz=0.277599999999996 0.241000195879143 0.0551000000000005 rpy=0 0 0, axis 0 1 0, limit lower=-0.524 upper=3.665 effort=50 velocity=1.57
- added joint right_rear_wheel_joint: type continuous, parent base_link, child right_back_wheel, origin xyz=0.156000000000004 0.219000195879132 0 rpy=0 0 0, axis 0 1 0
- added joint shoulder_pitch_joint: type revolute, parent big_course_part, child big_pitch_part, origin xyz=0 0.00320000000000144 0.0614876897975586 rpy=0 0 0, axis 0 -1 0, limit lower=-0.960 upper=1.571 effort=66 velocity=1.57
- added joint shoulder_yaw_joint: type revolute, parent base_link, child big_course_part, origin xyz=0.120249999999999 -0.00100019587899608 0.199849999999992 rpy=0 0 0, axis 0 0 1, limit lower=-2.356 upper=2.356 effort=66 velocity=1.57
- added joint wrist_pitch_joint: type revolute, parent small_pitch_part, child hands_pitch_part, origin xyz=0 0.0450999999999989 0.435999999999992 rpy=0 0 0, axis 0 1 0, limit lower=-1.57 upper=2.356 effort=6 velocity=1.57
- added joint wrist_roll_joint: type revolute, parent hands_pitch_part, child hands_roll_part, origin xyz=-0.0494999999999985 0.0265000000000013 0 rpy=0 0 0, axis -1 0 0, limit lower=-2.356 upper=2.356 effort=6 velocity=1.57
- added joint wrist_yaw_joint: type revolute, parent hands_roll_part, child handshands_course_part, origin xyz=-0.0265000000000413 0 0.0424999999999722 rpy=0 0 0, axis 0 0 -1, limit lower=-7.069 upper=7.069 effort=6 velocity=1.57
- joint lidar_joint: origin xyz=-0.1555 0.00100019587913144 0.300699999999992 rpy=0 0 0 -> xyz=-0.1555 0.0010002 0.3007 rpy=0 0 0

Commit message: car_urdf: sync arm axis directions from original urdf

File: car_urdf/urdf/car_urdf.urdf (robot description, URDF)
Before this commit: robot car_urdf, 21 links, 20 joints
Joints:
- joint elbow_pitch_joint: axis 0 -1 0 -> 0 1 0
- joint left_front_arm_joint: axis 0 -1 0 -> 0 1 0
- joint left_rear_arm_joint: axis 0 -1 0 -> 0 1 0
- joint shoulder_pitch_joint: axis 0 -1 0 -> 0 1 0
- joint wrist_yaw_joint: axis 0 0 -1 -> 0 0 1

Commit message: car_urdf: tune camera/depth frames and wheel simulation params

File: car_urdf/urdf/car_urdf.urdf (robot description, URDF)
Before this commit: robot car_urdf, 21 links, 20 joints
Links:
- added link catch_camera_optical_frame
Joints:
- added joint catch_camera_optical_joint: type fixed, parent catch_camera, child catch_camera_optical_frame, origin xyz=0 0 0 rpy=-1.5707963 0 -1.5707963
- joint gripper_camera_mount_joint: origin xyz=-0.0462233943895681 0.00134448857148927 0.0777106538096684 rpy=0 0 0 -> xyz=-0.0462233943895681 0.00134448857148927 0.0777106538096684 rpy=0 -1.5708 0

Commit message: fix(gazebo): stabilize gripper control and document troubleshooting

File: car_urdf/urdf/car_urdf.urdf (robot description, URDF)
Before this commit: robot car_urdf, 22 links, 21 joints
Joints:
- joint left_gripper_finger_joint: limit lower=-0.022 upper=0.03 effort=1 velocity=3 -> lower=-0.022 upper=0.03 effort=20 velocity=0.2
- joint right_gripper_finger_joint: limit lower=-0.022 upper=0.03 effort=1 velocity=3 -> lower=-0.022 upper=0.03 effort=20 velocity=0.2

Commit message: chore: checkpoint current simulation integration state

File: car_urdf/urdf/car_urdf.urdf (robot description, URDF)
Before this commit: robot car_urdf, 22 links, 21 joints
Links:
- link base_link: geometry collision box size=0.58 0.34 0.18; visual mesh filename=package://car_urdf/meshes/base_link.STL
- link left_ahead_wheel: geometry collision cylinder length=0.02 radius=0.029; visual mesh filename=package://car_urdf/meshes/left_ahead_wheel.STL
- link left_back_wheel: geometry collision cylinder length=0.02 radius=0.029; visual mesh filename=package://car_urdf/meshes/left_back_wheel.STL
- link right_ahead_wheel: geometry collision cylinder length=0.02 radius=0.029; visual mesh filename=package://car_urdf/meshes/right_ahead_wheel.STL
- link right_back_wheel: geometry collision cylinder length=0.02 radius=0.029; visual mesh filename=package://car_urdf/meshes/right_back_wheel.STL

Commit message: car_urdf: switch base sim to skid-steer wheel physics

File: car_urdf/urdf/car_urdf.urdf (robot description, URDF)
Before this commit: robot car_urdf, 22 links, 21 joints
Links:
- link left_ahead_wheel: mass 0.0487751853603894 -> 0.5
- link left_back_wheel: mass 0.0487751853603894 -> 0.5
- link right_ahead_wheel: mass 0.0487751853603893 -> 0.5
- link right_back_wheel: mass 0.0487751853603893 -> 0.5

Commit message: feat(car_urdf): update arm, gripper, and camera geometry

File: car_urdf/urdf/car_urdf.urdf (robot description, URDF)
Before this commit: robot car_urdf, 22 links, 21 joints
Links:
- link catch_camera: geometry visual mesh filename=package://car_urdf/meshes/catch-camera.STL
- link zhua1: geometry collision box size=0.001 0.0005 0.0025; visual mesh filename=package://car_urdf/meshes/zhualeft.STL
- link zhua2: geometry collision box size=0.001 0.0005 0.0025; visual mesh filename=package://car_urdf/meshes/zhuaright.STL
Joints:
- joint gripper_camera_mount_joint: origin xyz=-0.0462233943895681 0.00134448857148927 0.0777106538096684 rpy=0 -1.5708 0 -> xyz=-0.046223 0.0013445 0.073711 rpy=0 0 0
- joint left_gripper_finger_joint: origin xyz=0 0.021924 0.0985 rpy=0 0 0 -> xyz=0.00016784 -0.045039 0.1005 rpy=0 0 0
- joint right_gripper_finger_joint: origin xyz=-0.0038322 -0.021924 0.0985 rpy=0 0 0 -> xyz=0 0.045039 0.1005 rpy=0 0 0
- joint shoulder_yaw_joint: limit lower=-2.356 upper=2.356 effort=66 velocity=1.57 -> lower=-1 upper=1 effort=66 velocity=1.57
- joint wrist_pitch_joint: origin xyz=0 0.0450999999999989 0.435999999999992 rpy=0 0 0 -> xyz=0 0.0435999999999104 0.427999999999999 rpy=0 0 0
- joint wrist_roll_joint: origin xyz=-0.0494999999999985 0.0265000000000013 0 rpy=0 0 0 -> xyz=-0.0330007142673656 -0.0330000000000009 0.0530007142674829 rpy=0 0 0
- joint wrist_yaw_joint: origin xyz=-0.0265000000000413 0 0.0424999999999722 rpy=0 0 0 -> xyz=0.0330007142675045 0 0.0474000000000001 rpy=0 0 0

Commit message: car_urdf: checkpoint URDF updates

File: car_urdf/urdf/car_urdf.urdf (robot description, URDF)
Before this commit: robot car_urdf, 22 links, 21 joints
Links:
- added link camera_optical_frame
Joints:
- added joint camera_optical_joint: type fixed, parent camera, child camera_optical_frame, origin xyz=0 0 0 rpy=-1.5707963 0 -1.5707963
- joint gripper_camera_mount_joint: origin xyz=-0.046223 0.0013445 0.073711 rpy=0 0 0 -> xyz=-0.046223 0.0013445 0.073711 rpy=0 -1.5708 0

Commit message: car_urdf: add tool frames and rebase gripper geometry

File: car_urdf/urdf/car_urdf.urdf (robot description, URDF)
Before this commit: robot car_urdf, 23 links, 22 joints
Links:
- added link grasp_tcp
- added link tool0
Joints:
- added joint grasp_tcp_joint: type fixed, parent tool0, child grasp_tcp, origin xyz=0 0 0 rpy=0 0 0
- added joint tool0_joint: type fixed, parent handshands_course_part, child tool0, origin xyz=0.00008392 0 0.1075 rpy=0 0 0
- joint gripper_camera_mount_joint: origin xyz=-0.046223 0.0013445 0.073711 rpy=0 -1.5708 0 -> xyz=-0.04630692 0.0013445 -0.033789 rpy=0 -1.5708 0; parent handshands_course_part -> tool0
- joint left_gripper_finger_joint: axis 0 1 0 -> 0 -1 0; limit lower=-0.022 upper=0.03 effort=20 velocity=0.2 -> lower=0.0 upper=0.044 effort=20 velocity=0.2; origin xyz=0.00016784 -0.045039 0.1005 rpy=0 0 0 -> xyz=0.00008392 -0.023039 -0.007 rpy=0 0 0; parent handshands_course_part -> tool0
- joint right_gripper_finger_joint: axis 0 -1 0 -> 0 1 0; limit lower=-0.022 upper=0.03 effort=20 velocity=0.2 -> lower=0.0 upper=0.044 effort=20 velocity=0.2; origin xyz=0 0.045039 0.1005 rpy=0 0 0 -> xyz=-0.00008392 0.023039 -0.007 rpy=0 0 0; parent handshands_course_part -> tool0

Commit message: feat(car_urdf): add chassis and gripper control interfaces

File: car_urdf/urdf/car_urdf.urdf (robot description, URDF)
Before this commit: robot car_urdf, 25 links, 24 joints
Joints:
- joint left_rear_wheel_joint: mimic (none) -> joint=left_front_wheel_joint multiplier=1.0 offset=0.0
- joint right_rear_wheel_joint: mimic (none) -> joint=right_front_wheel_joint multiplier=1.0 offset=0.0

Commit message: urdf

File: car_urdf/urdf/car_urdf.urdf (robot description, URDF)
Before this commit: robot car_urdf, 19 links, 18 joints
Links:
- link base_link: geometry collision mesh filename=package://car_urdf/meshes/base_link.STL; visual mesh filename=package://car_urdf/meshes/base_link.STL
- link joint_1_link: geometry collision mesh filename=package://car_urdf/meshes/link1.STL; visual mesh filename=package://car_urdf/meshes/link1.STL
- link joint_2_link: geometry collision mesh filename=package://car_urdf/meshes/link2.STL; visual mesh filename=package://car_urdf/meshes/link2.STL
- link joint_3_link: geometry collision mesh filename=package://car_urdf/meshes/link3.STL; visual mesh filename=package://car_urdf/meshes/link3.STL
- link joint_4_link: geometry collision mesh filename=package://car_urdf/meshes/link4.STL; visual mesh filename=package://car_urdf/meshes/link4.STL
- link joint_5_link: geometry collision mesh filename=package://car_urdf/meshes/link5.STL; visual mesh filename=package://car_urdf/meshes/link5.STL
- link joint_6_link: geometry collision box size=0.16 0.06 0.06; visual box size=0.16 0.06 0.06
- link left_gripper_finger_link: geometry collision mesh filename=package://car_urdf/meshes/linkzhua1.STL; visual mesh filename=package://car_urdf/meshes/linkzhua1.STL
- link right_gripper_finger_link: geometry collision mesh filename=package://car_urdf/meshes/linkzhua2.STL; visual mesh filename=package://car_urdf/meshes/linkzhua2.STL
Joints:
- joint elbow_pitch_joint: axis 0 0 1 -> -1 0 0; origin (none) -> xyz=-0.0634554958516763 -0.08466955254996 0.44806252567829 rpy=0 0 0
- joint left_gripper_finger_joint: axis 0 1 0 -> -1 0 0; origin xyz=0.0 0.02 0.0 rpy=0 0 0 -> xyz=0 3.28514947361943 3.52837553837062 rpy=2.27424838462147 -0.821045734463187 1.57079632679491
- joint right_gripper_finger_joint: axis 0 -1 0 -> 0.789038133883824 0.605176450061446 -0.105736878940877; origin xyz=0.0 -0.02 0.0 rpy=0 0 0 -> xyz=0.00000000146632 -3.28527230451576 -3.52826115788185 rpy=2.12843991961849 -0.226127160063763 1.91590207174177
- joint shoulder_pitch_joint: axis 0 0 1 -> 1 0 0; origin (none) -> xyz=-0.0190610592148176 0.0037785921272299 0.492983162251151 rpy=0 0 0
- joint shoulder_yaw_joint: axis 0 0 1 -> -1 0 0; origin (none) -> xyz=0 -0.00419999972019724 0.054 rpy=-1.5707963267949 0 1.57030745170863
- joint wrist_pitch_joint: axis 0 0 1 -> 0 0 -1; origin (none) -> xyz=0.0867019191362518 -0.00673445031368503 -0.0154894931182463 rpy=-0.40986791242469 -0.000123856296620052 0
- joint wrist_roll_joint: axis 0 0 1 -> -1 0 0; origin (none) -> xyz=-0.00950565079420626 -0.0139732817540251 0.0866999999999829 rpy=1.5703914601342 0 0.973432793021899
- joint wrist_yaw_joint: origin (none) -> xyz=0.155699999999986 0 0 rpy=0 0 0
