Commit message: Align hybrid bringup and MoveIt configuration

File: car_moveit_config/config/car_urdf_gazebo.urdf (robot description, URDF)
Before this commit: robot oldcar111, 9 links, 8 joints
Links:
- removed link link1
- removed link link2
- removed link link3
- removed link link4
- removed link link5
- removed link linkzhua1
- removed link linkzhua2
- added link joint_1_link, mass 0.400617228197227; collision mesh filename=package://car_urdf/meshes/link1.STL; visual mesh filename=package://car_urdf/meshes/link1.STL
- added link joint_2_link, mass 0.230744553272649; collision mesh filename=package://car_urdf/meshes/link2.STL; visual mesh filename=package://car_urdf/meshes/link2.STL
- added link joint_3_link, mass 0.0824529162671332; collision mesh filename=package://car_urdf/meshes/link3.STL; visual mesh filename=package://car_urdf/meshes/link3.STL
- added link joint_4_link, mass 0.0824529142602831; collision mesh filename=package://car_urdf/meshes/link4.STL; visual mesh filename=package://car_urdf/meshes/link4.STL
- added link joint_5_link, mass 0.174467238698695; collision mesh filename=package://car_urdf/meshes/link5.STL; visual mesh filename=package://car_urdf/meshes/link5.STL
- added link joint_6_link, mass 0.001
- added link left_gripper_finger_link, mass 0.0276498547531941; visual mesh filename=package://car_urdf/meshes/linkzhua1.STL
- added link right_gripper_finger_link, mass 0.0276496025259502; visual mesh filename=package://car_urdf/meshes/linkzhua2.STL
- link base_link: geometry collision mesh filename=package://car_urdf/meshes/base_link.STL; visual mesh filename=package://car_urdf/meshes/base_link.STL
Joints:
- removed joint 1
- removed joint 2
- removed joint 3
- removed joint 4
- removed joint 5
- removed joint zhua1
- removed joint zhua2
- added joint elbow_pitch_joint: type continuous, parent joint_2_link, child joint_3_link, origin xyz=-0.0634554958516763 -0.08466955254996 0.44806252567829 rpy=0 0 0, axis -1 0 0
- added joint left_gripper_finger_joint: type prismatic, parent joint_6_link, child left_gripper_finger_link, origin xyz=0.0 0.02 0.0 rpy=0 0 0, axis 0 1 0, limit lower=-0.06 upper=0 effort=100 velocity=0.2
- added joint right_gripper_finger_joint: type fixed, parent joint_6_link, child right_gripper_finger_link, origin xyz=0.0 -0.02 0.0 rpy=0 0 0
- added joint shoulder_pitch_joint: type revolute, parent joint_1_link, child joint_2_link, origin xyz=-0.0190610592148176 0.0037785921272299 0.492983162251151 rpy=0 0 0, axis 1 0 0, limit lower=-2.93 upper=2.95 effort=0 velocity=0
- added joint shoulder_yaw_joint: type revolute, parent base_link, child joint_1_link, origin xyz=0 -0.00419999972019724 0.054 rpy=-1.5707963267949 0 1.57030745170863, axis -1 0 0, limit lower=-3.14 upper=0 effort=0 velocity=0
- added joint wrist_pitch_joint: type continuous, parent joint_3_link, child joint_4_link, origin xyz=0.0867019191362518 -0.00673445031368503 -0.0154894931182463 rpy=-0.40986791242469 -0.000123856296620052 0, axis 0 0 -1
- added joint wrist_roll_joint: type continuous, parent joint_4_link, child joint_5_link, origin xyz=-0.00950565079420626 -0.0139732817540251 0.0866999999999829 rpy=1.5703914601342 0 0.973432793021899, axis -1 0 0
- added joint wrist_yaw_joint: type continuous, parent joint_5_link, child joint_6_link, origin xyz=0 0 0 rpy=0 0 0, axis 0 0 1

File: car_urdf/urdf/car_urdf.urdf (robot description, URDF)
Before this commit: robot car_urdf, 19 links, 18 joints
Joints:
- joint left_gripper_finger_joint: limit lower=-0.06 upper=0.0 effort=100 velocity=0.2 -> lower=4.748646 upper=4.808646 effort=100 velocity=0.2
- joint right_gripper_finger_joint: limit lower=-0.06 upper=0.0 effort=100 velocity=0.2 -> lower=4.748646 upper=4.808646 effort=100 velocity=0.2
